File: PCB/main/main.kicad_sch (KiCad schematic)
At the start: 4 parts, among them J1 Conn_01x33_Female, J2 Conn_01x33_Female, J3 Conn_01x33_Female, J4 Conn_01x33_Female

Commit message: changes made to all
Other:
- note removed: "Useful to watch: https://www.youtube.com/watch?v=gGix1oYhTRs"
