File: PCB/main/main.kicad_sch (KiCad schematic)
At the start: 4 parts, among them J1 Conn_01x33_Female, J2 Conn_01x33_Female, J3 Conn_01x33_Female, J4 Conn_01x33_Female

Commit message: created BOM
Parts:
- J2, J3: LCSC C1234 (example) -> (none)
Changed lines of the file:
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@@
       (effects (font (size 1.27 1.27)) hide)
     )
-    (property "LCSC" "C1234 (example)" (id 4) (at 224.155 64.77 0)
+    (property "LCSC" "" (id 4) (at 224.155 64.77 0)
       (effects (font (size 1.27 1.27)) hide)
     )
@@
       (effects (font (size 1.27 1.27)) hide)
     )
-    (property "LCSC" "C1234 (example)" (id 4) (at 243.205 64.77 0)
+    (property "LCSC" "" (id 4) (at 243.205 64.77 0)
       (effects (font (size 1.27 1.27)) hide)
     )
