File: PCB/main/power.kicad_sch (KiCad schematic)
At the start: 22 parts, among them J1 47346-0001, Q1 IRF9540NPbF, U1 MCP73831-2-OT, U2 FT232RL, U3 MCP1700-3302E_TO92

Commit message: git main schematics updated
Parts:
- J5: renamed from J1; footprint SamacSys_Parts:47346-0001 -> SamacSys_Parts_Power:47346-0001
- renumbered C5 to C1, C6 to C2, C1 to C3, C2 to C4, C7 to C5, C8 to C6, C3 to C7, C4 to C8, D3 to D2, D2 to D3, R4 to R3
Connections:
- net Earth renamed GND
