File: PCB/main/power.kicad_sch (KiCad schematic)
At the start: 25 parts, among them IC4 TP4056-42-ESOP8, J10 PZ254V-11-02P, J11 ICH-340-CTT, J5 47346-0001, J6 PZ254V-11-02P, J7 PZ254V-11-02P, J8 MTP125-1103S1, Q1 AO3401A, U1 HT75xx-1-SOT89

Commit message: NEW PCB ADDED
Parts:
- C2, C6, C7, C8: Comment (none) -> 10uF; LCSC (none) -> C13585
- C5: Comment (none) -> 100nF; LCSC (none) -> C1790
- D1, D2: Comment (none) -> diode; LCSC (none) -> C2480
- IC4: Comment (none) -> ESOP-8 Battery Management ICs ROHS; LCSC (none) -> C16581
- J10: footprint SamacSys_Parts_Power:HDRV2W64P0X254_1X2_508X250X873P -> SamacSys_Parts:HDRV2W64P0X254_1X2_508X250X873P; Comment (none) -> pin header (2x1); LCSC (none) -> C492401
- J11: Comment (none) -> Transceiver 2Mbps USB 2.0 SOP-16_150mil USB ICs ROHS; LCSC (none) -> C84681
- J5: footprint SamacSys_Parts_Microcontroller:47346-0001 -> SamacSys_Parts:47346-0001
- J6, J7: footprint SamacSys_Parts_Power:HDRV2W64P0X254_1X2_508X250X873P -> SamacSys_Parts:HDRV2W64P0X254_1X2_508X250X873P; Comment 2 pin male header -> pin header (2x1)
- J8: footprint SamacSys_Parts_Power:HDRV3W64P0X254_1X3_762X250X885P -> SamacSys_Parts:HDRV3W64P0X254_1X3_762X250X885P; Comment 3 pin male header -> pin header (3x1)
- LED1, LED2: Comment (none) -> LED_0603; LCSC (none) -> C72043
- Q1: Comment (none) -> 30V 4A 44mΩ@10V,4.3A 1.4W 1.3V@250μA P Channel SOT-23-3L MO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; LCSC (none) -> C15127
- R1: footprint RESC1608X55N -> SamacSys_Parts:RESC1608X55N; Comment (none) -> 1.2k; LCSC (none) -> C22765
Changed lines of the file:
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@@
       (effects (font (size 1.27 1.27)) (justify left) hide)
+    )
+    (property "Comment" "10uF" (id 12) (at 150.495 120.015 0)
+      (effects (font (size 1.27 1.27)) hide)
+    )
+    (property "LCSC" "C13585" (id 13) (at 150.495 120.015 0)
+      (effects (font (size 1.27 1.27)) hide)
     )
     (pin "1")
@@
       (effects (font (size 1.27 1.27)) (justify left) hide)
     )
+    (property "Comment" "10uF" (id 12) (at 264.16 116.84 0)
+      (effects (font (size 1.27 1.27)) hide)
+    )
+    (property "LCSC" "C13585" (id 13) (at 264.16 116.84 0)
+      (effects (font (size 1.27 1.27)) hide)
+    )
     (pin "1")
     (pin "2")
@@
     (property "Arrow Price/Stock" "https://www.arrow.com/en/products/cl21c101jbannnc/samsung-electro-mechanics?region=nac" (id 11) (at 114.3 107.315 0)
       (effects (font (size 1.27 1.27)) (justify left) hide)
+    )
+    (property "Comment" "100nF" (id 12) (at 92.71 116.205 0)
+      (effects (font (size 1.27 1.27)) hide)
+    )
+    (property "LCSC" "C1790" (id 13) (at 92.71 116.205 0)
+      (effects (font (size 1.27 1.27)) hide)
     )
     (pin "1")
@@
       (effects (font (size 1.27 1.27)) (justify left))
     )
-    (property "Footprint" "SamacSys_Parts_Power:HDRV2W64P0X254_1X2_508X250X873P" (id 2) (at 171.45 161.29 0)
+    (property "Footprint" "SamacSys_Parts:HDRV2W64P0X254_1X2_508X250X873P" (id 2) (at 171.45 161.29 0)
       (effects (font (size 1.27 1.27)) (justify left) hide)
     )
@@
       (effects (font (size 1.27 1.27)) (justify left) hide)
     )
-    (property "Comment" "2 pin male header" (id 12) (at 168.91 144.78 0)
+    (property "Comment" "pin header (2x1)" (id 12) (at 168.91 144.78 0)
       (effects (font (size 1.27 1.27)) hide)
     )
@@
       (effects (font (size 1.27 1.27)) (justify left bottom) hide)
     )
+    (property "Comment" "LED_0603" (id 12) (at 144.145 72.39 0)
+      (effects (font (size 1.27 1.27)) hide)
+    )
+    (property "LCSC" "C72043" (id 13) (at 144.145 72.39 0)
+      (effects (font (size 1.27 1.27)) hide)
+    )
     (pin "1")
     (pin "2")
@@
     (property "Arrow Price/Stock" "" (id 11) (at 60.96 153.035 0)
       (effects (font (size 1.27 1.27)) (justify left) hide)
+    )
+    (property "Comment" "Transceiver 2Mbps USB 2.0 SOP-16_150mil USB ICs ROHS" (id 12) (at 41.91 132.715 0)
+      (effects (font (size 1.27 1.27)) hide)
+    )
+    (property "LCSC" "C84681" (id 13) (at 41.91 132.715 0)
+      (effects (font (size 1.27 1.27)) hide)
     )
     (pin "1")
@@
       (effects (font (size 1.27 1.27)) (justify left))
     )
-    (property "Footprint" "SamacSys_Parts_Power:HDRV3W64P0X254_1X3_762X250X885P" (id 2) (at 217.17 118.11 0)
+    (property "Footprint" "SamacSys_Parts:HDRV3W64P0X254_1X3_762X250X885P" (id 2) (at 217.17 118.11 0)
       (effects (font (size 1.27 1.27)) (justify left) hide)
     )
@@
       (effects (font (size 1.27 1.27)) (justify left) hide)
     )
-    (property "Comment" "3 pin male header" (id 12) (at 214.63 101.6 0)
+    (property "Comment" "pin header (3x1)" (id 12) (at 214.63 101.6 0)
       (effects (font (size 1.27 1.27)) hide)
     )
@@
       (effects (font (size 1.27 1.27)) (justify left) hide)
     )
+    (property "Comment" "10uF" (id 12) (at 23.495 183.515 0)
+      (effects (font (size 1.27 1.27)) hide)
+    )
+    (property "LCSC" "C13585" (id 13) (at 23.495 183.515 0)
+      (effects (font (size 1.27 1.27)) hide)
+    )
     (pin "1")
     (pin "2")
@@
     (property "Reference" "J5" (id 0) (at 64.135 60.96 90))
     (property "Value" "47346-0001" (id 1) (at 64.135 63.5 90))
-    (property "Footprint" "SamacSys_Parts_Microcontroller:47346-0001" (id 2) (at 57.785 64.77 0)
+    (property "Footprint" "SamacSys_Parts:47346-0001" (id 2) (at 57.785 64.77 0)
       (effects (font (size 1.27 1.27)) (justify left) hide)
     )
@@
     (property "Arrow Price/Stock" "https://www.arrow.com/en/products/cl31a106kbhnnne/samsung-electro-mechanics?region=nac" (id 11) (at 249.555 108.585 0)
       (effects (font (size 1.27 1.27)) (justify left) hide)
+    )
+    (property "Comment" "10uF" (id 12) (at 227.965 117.475 0)
+      (effects (font (size 1.27 1.27)) hide)
+    )
+    (property "LCSC" "C13585" (id 13) (at 227.965 117.475 0)
+      (effects (font (size 1.27 1.27)) hide)
     )
     (pin "1")
@@
       (effects (font (size 1.27 1.27)) (justify left bottom) hide)
     )
+    (property "Comment" "LED_0603" (id 12) (at 121.92 79.375 0)
+      (effects (font (size 1.27 1.27)) hide)
+    )
+    (property "LCSC" "C72043" (id 13) (at 121.92 79.375 0)
+      (effects (font (size 1.27 1.27)) hide)
+    )
     (pin "1")
     (pin "2")
@@
       (effects (font (size 1.27 1.27)) (justify left) hide)
     )
+    (property "Comment" "diode" (id 12) (at 207.01 101.6 0)
+      (effects (font (size 1.27 1.27)) hide)
+    )
+    (property "LCSC" "C2480" (id 13) (at 207.01 101.6 0)
+      (effects (font (size 1.27 1.27)) hide)
+    )
     (pin "1")
     (pin "2")
@@
       (effects (font (size 1.27 1.27)) (justify right))
     )
-    (property "Footprint" "RESC1608X55N" (id 2) (at 100.33 116.205 0)
+    (property "Footprint" "SamacSys_Parts:RESC1608X55N" (id 2) (at 100.33 116.205 0)
       (effects (font (size 1.27 1.27)) (justify left) hide)
     )
@@
     (property "Arrow Price/Stock" "" (id 11) (at 123.19 116.205 0)
       (effects (font (size 1.27 1.27)) (justify left) hide)
+    )
+    (property "Comment" "1.2k" (id 12) (at 101.6 130.175 0)
+      (effects (font (size 1.27 1.27)) hide)
+    )
+    (property "LCSC" "C22765" (id 13) (at 101.6 130.175 0)
+      (effects (font (size 1.27 1.27)) hide)
     )
     (pin "1")
@@
     (property "Arrow Price/Stock" "" (id 11) (at 144.145 114.3 0)
       (effects (font (size 1.27 1.27)) (justify left) hide)
+    )
+    (property "Comment" "ESOP-8 Battery Management ICs ROHS" (id 12) (at 117.475 93.98 0)
+      (effects (font (size 1.27 1.27)) hide)
+    )
+    (property "LCSC" "C16581" (id 13) (at 117.475 93.98 0)
+      (effects (font (size 1.27 1.27)) hide)
     )
     (pin "1")
@@
       (effects (font (size 1.27 1.27)) (justify right))
     )
-    (property "Footprint" "SamacSys_Parts_Power:HDRV2W64P0X254_1X2_508X250X873P" (id 2) (at 163.83 125.73 0)
+    (property "Footprint" "SamacSys_Parts:HDRV2W64P0X254_1X2_508X250X873P" (id 2) (at 163.83 125.73 0)
       (effects (font (size 1.27 1.27)) (justify left) hide)
     )
@@
       (effects (font (size 1.27 1.27)) (justify left) hide)
     )
-    (property "Comment" "2 pin male header" (id 12) (at 166.37 142.24 0)
+    (property "Comment" "pin header (2x1)" (id 12) (at 166.37 142.24 0)
       (effects (font (size 1.27 1.27)) hide)
     )
@@
     (property "Arrow Price/Stock" "https://www.arrow.com/en/products/ss14/on-semiconductor?region=nac" (id 11) (at 227.965 75.565 0)
       (effects (font (size 1.27 1.27)) (justify left) hide)
+    )
+    (property "Comment" "diode" (id 12) (at 208.915 88.265 0)
+      (effects (font (size 1.27 1.27)) hide)
+    )
+    (property "LCSC" "C2480" (id 13) (at 208.915 88.265 0)
+      (effects (font (size 1.27 1.27)) hide)
     )
     (pin "1")
@@
       (effects (font (size 1.27 1.27)) (justify left) hide)
     )
+    (property "Comment" "30V 4A 44mΩ@10V,4.3A 1.4W 1.3V@250μA P Channel SOT-23-3L MOSFETs ROHS" (id 12) (at 177.165 93.98 0)
+      (effects (font (size 1.27 1.27)) hide)
+    )
+    (property "LCSC" "C15127" (id 13) (at 177.165 93.98 0)
+      (effects (font (size 1.27 1.27)) hide)
+    )
     (pin "1")
     (pin "2")
@@
       (effects (font (size 1.27 1.27)) (justify left))
     )
-    (property "Footprint" "SamacSys_Parts_Power:HDRV2W64P0X254_1X2_508X250X873P" (id 2) (at 174.625 107.95 0)
+    (property "Footprint" "SamacSys_Parts:HDRV2W64P0X254_1X2_508X250X873P" (id 2) (at 174.625 107.95 0)
       (effects (font (size 1.27 1.27)) (justify left) hide)
     )
@@
       (effects (font (size 1.27 1.27)) (justify left) hide)
     )
-    (pin "1")
+    (property "Comment" "pin header (2x1)" (id 12) (at 158.115 110.49 0)
+      (effects (font (size 1.27 1.27)) hide)
+    )
+    (property "LCSC" "C492401" (id 13) (at 158.115 110.49 0)
+      (effects (font (size 1.27 1.27)) hide)
+    )
+    (pin "1")
