File: PCB/main/microcontroller_interfacing.kicad_sch (KiCad schematic)
At the start: 9 parts, among them IC2 LM358DT, IC3 AT24C256C-SSHL-T

Commit message: added test points and jumpers
Parts:
- removed TP? (x2): TestPoint, symbol Connector:TestPoint
- added TP5, TP6: 5017, SamacSys_Parts:5017, symbol SamacSys_Parts_power:5017
Connections:
- net +3v3: now also TP6.1
- net -3v3: now also TP5.1
Changed lines of the file:
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@@
   (junction (at 78.74 68.58) (diameter 0) (color 0 0 0 0)
   )
+  (junction (at 121.92 73.66) (diameter 0) (color 0 0 0 0)
+  )
   (junction (at 104.14 128.27) (diameter 0) (color 0 0 0 0)
   )
@@
   )
   (junction (at 185.42 120.65) (diameter 0) (color 0 0 0 0)
+  )
+  (junction (at 92.71 66.04) (diameter 0) (color 0 0 0 0)
   )
   (junction (at 182.88 120.65) (diameter 0) (color 0 0 0 0)
@@
     (stroke (width 0) (type default) (color 0 0 0 0))
   )
+  (wire (pts (xy 121.92 73.66) (xy 125.73 73.66))
+    (stroke (width 0) (type default) (color 0 0 0 0))
+  )
+  (wire (pts (xy 90.17 66.04) (xy 92.71 66.04))
+    (stroke (width 0) (type default) (color 0 0 0 0))
+  )
   (wire (pts (xy 31.75 68.58) (xy 39.37 68.58))
     (stroke (width 0) (type default) (color 0 0 0 0))
@@
     (stroke (width 0) (type default) (color 0 0 0 0))
   )
+  (wire (pts (xy 92.71 66.04) (xy 93.98 66.04))
+    (stroke (width 0) (type default) (color 0 0 0 0))
+  )
   (wire (pts (xy 59.69 85.09) (xy 59.69 86.36))
     (stroke (width 0) (type default) (color 0 0 0 0))
@@
     (stroke (width 0) (type default) (color 0 0 0 0))
   )
-  (wire (pts (xy 121.92 73.66) (xy 125.73 73.66))
-    (stroke (width 0) (type default) (color 0 0 0 0))
-  )
   (wire (pts (xy 148.59 91.44) (xy 148.59 99.06))
     (stroke (width 0) (type default) (color 0 0 0 0))
@@
   )
   (wire (pts (xy 182.88 33.02) (xy 182.88 38.1))
-    (stroke (width 0) (type default) (color 0 0 0 0))
-  )
-  (wire (pts (xy 90.17 66.04) (xy 93.98 66.04))
     (stroke (width 0) (type default) (color 0 0 0 0))
   )
@@
   )
   (text "Sallen-Key LPF Filter for noise reduction\nand also maintain ADC accuracy\n"
-    (at 80.01 53.34 0)
+    (at 78.74 44.45 0)
     (effects (font (size 1.27 1.27)) (justify left bottom))
   )
@@
     (pin "1")
     (pin "2")
+  )
+  (symbol (lib_id "SamacSys_Parts_power:5017") (at 92.71 66.04 90) (unit 1)
+    (in_bom yes) (on_board yes) (fields_autoplaced)
+    (property "Reference" "TP5" (id 0) (at 96.52 54.6099 90)
+      (effects (font (size 1.27 1.27)) (justify right))
+    )
+    (property "Value" "5017" (id 1) (at 96.52 57.1499 90)
+      (effects (font (size 1.27 1.27)) (justify right))
+    )
+    (property "Footprint" "SamacSys_Parts:5017" (id 2) (at 90.17 49.53 0)
+      (effects (font (size 1.27 1.27)) (justify left) hide)
+    )
+    (property "Datasheet" "http://www.keyelco.com/product.cfm/product_id/1355" (id 3) (at 92.71 49.53 0)
+      (effects (font (size 1.27 1.27)) (justify left) hide)
+    )
+    (property "Description" "KEYSTONE - 5017 - TEST POINT, PCB, MINIATURE, SMT" (id 4) (at 95.25 49.53 0)
+      (effects (font (size 1.27 1.27)) (justify left) hide)
+    )
+    (property "Height" "" (id 5) (at 97.79 49.53 0)
+      (effects (font (size 1.27 1.27)) (justify left) hide)
+    )
+    (property "Manufacturer_Name" "Keystone Electronics" (id 6) (at 100.33 49.53 0)
+      (effects (font (size 1.27 1.27)) (justify left) hide)
+    )
+    (property "Manufacturer_Part_Number" "5017" (id 7) (at 102.87 49.53 0)
+      (effects (font (size 1.27 1.27)) (justify left) hide)
+    )
+    (property "Mouser Part Number" "534-5017" (id 8) (at 105.41 49.53 0)
+      (effects (font (size 1.27 1.27)) (justify left) hide)
+    )
+    (property "Mouser Price/Stock" "https://www.mouser.co.uk/ProductDetail/Keystone-Electronics/5017?qs=Rc9fedAPY0Oq34lsnTvuLg%3D%3D" (id 9) (at 107.95 49.53 0)
+      (effects (font (size 1.27 1.27)) (justify left) hide)
+    )
+    (property "Arrow Part Number" "" (id 10) (at 110.49 49.53 0)
+      (effects (font (size 1.27 1.27)) (justify left) hide)
+    )
+    (property "Arrow Price/Stock" "" (id 11) (at 113.03 49.53 0)
+      (effects (font (size 1.27 1.27)) (justify left) hide)
+    )
+    (pin "1")
   )
   (symbol (lib_id "SamacSys_Parts_Microcontroller:RC0603FR-071KL") (at 60.96 59.69 0) (unit 1)
@@
     (pin "1")
   )
+  (symbol (lib_id "SamacSys_Parts_power:5017") (at 121.92 73.66 270) (unit 1)
+    (in_bom yes) (on_board yes) (fields_autoplaced)
+    (property "Reference" "TP6" (id 0) (at 125.73 82.5499 90)
+      (effects (font (size 1.27 1.27)) (justify left))
+    )
+    (property "Value" "5017" (id 1) (at 125.73 85.0899 90)
+      (effects (font (size 1.27 1.27)) (justify left))
+    )
+    (property "Footprint" "SamacSys_Parts:5017" (id 2) (at 124.46 90.17 0)
+      (effects (font (size 1.27 1.27)) (justify left) hide)
+    )
+    (property "Datasheet" "http://www.keyelco.com/product.cfm/product_id/1355" (id 3) (at 121.92 90.17 0)
+      (effects (font (size 1.27 1.27)) (justify left) hide)
+    )
+    (property "Description" "KEYSTONE - 5017 - TEST POINT, PCB, MINIATURE, SMT" (id 4) (at 119.38 90.17 0)
+      (effects (font (size 1.27 1.27)) (justify left) hide)
+    )
+    (property "Height" "" (id 5) (at 116.84 90.17 0)
+      (effects (font (size 1.27 1.27)) (justify left) hide)
+    )
+    (property "Manufacturer_Name" "Keystone Electronics" (id 6) (at 114.3 90.17 0)
+      (effects (font (size 1.27 1.27)) (justify left) hide)
+    )
+    (property "Manufacturer_Part_Number" "5017" (id 7) (at 111.76 90.17 0)
+      (effects (font (size 1.27 1.27)) (justify left) hide)
+    )
+    (property "Mouser Part Number" "534-5017" (id 8) (at 109.22 90.17 0)
+      (effects (font (size 1.27 1.27)) (justify left) hide)
+    )
+    (property "Mouser Price/Stock" "https://www.mouser.co.uk/ProductDetail/Keystone-Electronics/5017?qs=Rc9fedAPY0Oq34lsnTvuLg%3D%3D" (id 9) (at 106.68 90.17 0)
+      (effects (font (size 1.27 1.27)) (justify left) hide)
+    )
+    (property "Arrow Part Number" "" (id 10) (at 104.14 90.17 0)
+      (effects (font (size 1.27 1.27)) (justify left) hide)
+    )
+    (property "Arrow Price/Stock" "" (id 11) (at 101.6 90.17 0)
+      (effects (font (size 1.27 1.27)) (justify left) hide)
+    )
+    (pin "1")
+  )
   (symbol (lib_id "power:GND") (at 182.88 124.46 0) (unit 1)
     (in_bom yes) (on_board yes) (fields_autoplaced)
@@
     )
     (property "Datasheet" "" (id 3) (at 182.88 124.46 0)
-      (effects (font (size 1.27 1.27)) hide)
-    )
-    (pin "1")
-  )
-  (symbol (lib_id "Connector:TestPoint") (at 92.71 66.04 0) (unit 1)
-    (in_bom yes) (on_board yes) (fields_autoplaced)
-    (property "Reference" "TP?" (id 0) (at 95.25 61.4679 0)
-      (effects (font (size 1.27 1.27)) (justify left))
-    )
-    (property "Value" "TestPoint" (id 1) (at 95.25 64.0079 0)
-      (effects (font (size 1.27 1.27)) (justify left))
-    )
-    (property "Footprint" "" (id 2) (at 97.79 66.04 0)
-      (effects (font (size 1.27 1.27)) hide)
-    )
-    (property "Datasheet" "~" (id 3) (at 97.79 66.04 0)
       (effects (font (size 1.27 1.27)) hide)
     )
@@
     (pin "2")
   )
-  (symbol (lib_id "Connector:TestPoint") (at 124.46 73.66 180) (unit 1)
-    (in_bom yes) (on_board yes) (fields_autoplaced)
-    (property "Reference" "TP?" (id 0) (at 127 75.6919 0)
-      (effects (font (size 1.27 1.27)) (justify right))
-    )
-    (property "Value" "TestPoint" (id 1) (at 127 78.2319 0)
-      (effects (font (size 1.27 1.27)) (justify right))
-    )
-    (property "Footprint" "" (id 2) (at 119.38 73.66 0)
-      (effects (font (size 1.27 1.27)) hide)
-    )
-    (property "Datasheet" "~" (id 3) (at 119.38 73.66 0)
-      (effects (font (size 1.27 1.27)) hide)
-    )
-    (pin "1")
-  )
   (symbol (lib_id "SamacSys_Parts_Microcontroller:AT24C256C-SSHL-T") (at 110.49 125.73 0) (unit 1)

Commit message: gerber files and dat
Parts:
- added C13: CC0603KRX7R9BB104, CAPC1608X90N, symbol SamacSys_Parts_Power:CC0603KRX7R9BB104
- added J9: PZ254V-11-02P, HDRV2W64P0X254_1X2_508X250X873P, symbol SamacSys_Parts_Power:PZ254V-11-02P
- renumbered TP5 to TP8, TP6 to TP9
Connections:
- net GND: now also C13.2, J9.2
- net Vsupply: no longer MCU1.7 (NRST)
- new net: C13.1, J9.1, MCU1.7 (NRST)
Changed lines of the file:
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@@
   (junction (at 185.42 33.02) (diameter 0) (color 0 0 0 0)
+  )
+  (junction (at 223.52 43.18) (diameter 0) (color 0 0 0 0)
   )
   (junction (at 110.49 133.35) (diameter 0) (color 0 0 0 0)
@@
     (stroke (width 0) (type default) (color 0 0 0 0))
   )
+  (wire (pts (xy 237.49 25.4) (xy 223.52 25.4))
+    (stroke (width 0) (type default) (color 0 0 0 0))
+  )
   (wire (pts (xy 104.14 128.27) (xy 110.49 128.27))
     (stroke (width 0) (type default) (color 0 0 0 0))
@@
     (stroke (width 0) (type default) (color 0 0 0 0))
   )
+  (wire (pts (xy 223.52 43.18) (xy 236.22 43.18))
+    (stroke (width 0) (type default) (color 0 0 0 0))
+  )
   (wire (pts (xy 104.14 130.81) (xy 110.49 130.81))
     (stroke (width 0) (type default) (color 0 0 0 0))
@@
     (stroke (width 0) (type default) (color 0 0 0 0))
   )
+  (wire (pts (xy 236.22 45.72) (xy 234.95 45.72))
+    (stroke (width 0) (type default) (color 0 0 0 0))
+  )
   (wire (pts (xy 148.59 99.06) (xy 170.18 99.06))
     (stroke (width 0) (type default) (color 0 0 0 0))
@@
     (stroke (width 0) (type default) (color 0 0 0 0))
   )
-  (wire (pts (xy 200.66 43.18) (xy 207.01 43.18))
+  (wire (pts (xy 200.66 43.18) (xy 223.52 43.18))
     (stroke (width 0) (type default) (color 0 0 0 0))
   )
@@
   )
   (wire (pts (xy 182.88 33.02) (xy 182.88 38.1))
+    (stroke (width 0) (type default) (color 0 0 0 0))
+  )
+  (wire (pts (xy 234.95 45.72) (xy 234.95 52.07))
+    (stroke (width 0) (type default) (color 0 0 0 0))
+  )
+  (wire (pts (xy 223.52 39.37) (xy 223.52 43.18))
+    (stroke (width 0) (type default) (color 0 0 0 0))
+  )
+  (wire (pts (xy 223.52 25.4) (xy 223.52 26.67))
     (stroke (width 0) (type default) (color 0 0 0 0))
   )
@@
   (label "OUT1" (at 163.83 78.74 180)
     (effects (font (size 1.27 1.27)) (justify right bottom))
-  )
-  (global_label "Vsupply" (shape input) (at 207.01 43.18 0) (fields_autoplaced)
-    (effects (font (size 1.27 1.27)) (justify left))
-    (property "Intersheet References" "${INTERSHEET_REFS}" (id 0) (at 216.6198 43.1006 0)
-      (effects (font (size 1.27 1.27)) (justify left) hide)
-    )
   )
   (global_label "USART1_RX" (shape input) (at 142.24 101.6 180) (fields_autoplaced)
@@
     (pin "2")
   )
+  (symbol (lib_id "power:GND") (at 237.49 25.4 90) (unit 1)
+    (in_bom yes) (on_board yes) (fields_autoplaced)
+    (property "Reference" "#PWR041" (id 0) (at 243.84 25.4 0)
+      (effects (font (size 1.27 1.27)) hide)
+    )
+    (property "Value" "GND" (id 1) (at 241.3 25.3999 90)
+      (effects (font (size 1.27 1.27)) (justify right))
+    )
+    (property "Footprint" "" (id 2) (at 237.49 25.4 0)
+      (effects (font (size 1.27 1.27)) hide)
+    )
+    (property "Datasheet" "" (id 3) (at 237.49 25.4 0)
+      (effects (font (size 1.27 1.27)) hide)
+    )
+    (pin "1")
+  )
   (symbol (lib_id "SamacSys_Parts_power:5017") (at 92.71 66.04 90) (unit 1)
     (in_bom yes) (on_board yes) (fields_autoplaced)
-    (property "Reference" "TP5" (id 0) (at 96.52 54.6099 90)
+    (property "Reference" "TP8" (id 0) (at 96.52 54.6099 90)
       (effects (font (size 1.27 1.27)) (justify right))
     )
@@
   (symbol (lib_id "power:PWR_FLAG") (at 110.49 137.16 180) (unit 1)
     (in_bom yes) (on_board yes) (fields_autoplaced)
-    (property "Reference" "#FLG0103" (id 0) (at 110.49 139.065 0)
+    (property "Reference" "#FLG07" (id 0) (at 110.49 139.065 0)
       (effects (font (size 1.27 1.27)) hide)
     )
@@
     (pin "1")
   )
+  (symbol (lib_id "power:GND") (at 234.95 52.07 0) (unit 1)
+    (in_bom yes) (on_board yes) (fields_autoplaced)
+    (property "Reference" "#PWR040" (id 0) (at 234.95 58.42 0)
+      (effects (font (size 1.27 1.27)) hide)
+    )
+    (property "Value" "GND" (id 1) (at 234.95 57.15 0))
+    (property "Footprint" "" (id 2) (at 234.95 52.07 0)
+      (effects (font (size 1.27 1.27)) hide)
+    )
+    (property "Datasheet" "" (id 3) (at 234.95 52.07 0)
+      (effects (font (size 1.27 1.27)) hide)
+    )
+    (pin "1")
+  )
   (symbol (lib_id "SamacSys_Parts_power:5017") (at 121.92 73.66 270) (unit 1)
     (in_bom yes) (on_board yes) (fields_autoplaced)
-    (property "Reference" "TP6" (id 0) (at 125.73 82.5499 90)
+    (property "Reference" "TP9" (id 0) (at 125.73 82.5499 90)
       (effects (font (size 1.27 1.27)) (justify left))
     )
@@
   (symbol (lib_id "power:GND") (at 182.88 124.46 0) (unit 1)
     (in_bom yes) (on_board yes) (fields_autoplaced)
-    (property "Reference" "#PWR040" (id 0) (at 182.88 130.81 0)
+    (property "Reference" "#PWR038" (id 0) (at 182.88 130.81 0)
       (effects (font (size 1.27 1.27)) hide)
     )
@@
     (pin "1")
   )
+  (symbol (lib_id "SamacSys_Parts_Power:PZ254V-11-02P") (at 236.22 43.18 0) (unit 1)
+    (in_bom yes) (on_board yes) (fields_autoplaced)
+    (property "Reference" "J9" (id 0) (at 252.73 43.1799 0)
+      (effects (font (size 1.27 1.27)) (justify left))
+    )
+    (property "Value" "PZ254V-11-02P" (id 1) (at 252.73 45.7199 0)
+      (effects (font (size 1.27 1.27)) (justify left))
+    )
+    (property "Footprint" "HDRV2W64P0X254_1X2_508X250X873P" (id 2) (at 252.73 40.64 0)
+      (effects (font (size 1.27 1.27)) (justify left) hide)
+    )
+    (property "Datasheet" "https://datasheet.lcsc.com/lcsc/2003141409_XFCN-PZ254V-11-02P_C492401.pdf" (id 3) (at 252.73 43.18 0)
+      (effects (font (size 1.27 1.27)) (justify left) hide)
+    )
+    (property "Description" "Straight 1 2 2.54mm Black Brass Plugin,P=2.54mm Pin Headers ROHS" (id 4) (at 252.73 45.72 0)
+      (effects (font (size 1.27 1.27)) (justify left) hide)
+    )
+    (property "Height" "8.73" (id 5) (at 252.73 48.26 0)
+      (effects (font (size 1.27 1.27)) (justify left) hide)
+    )
+    (property "Manufacturer_Name" "XFCN" (id 6) (at 252.73 50.8 0)
+      (effects (font (size 1.27 1.27)) (justify left) hide)
+    )
+    (property "Manufacturer_Part_Number" "PZ254V-11-02P" (id 7) (at 252.73 53.34 0)
+      (effects (font (size 1.27 1.27)) (justify left) hide)
+    )
+    (property "Mouser Part Number" "" (id 8) (at 252.73 55.88 0)
+      (effects (font (size 1.27 1.27)) (justify left) hide)
+    )
+    (property "Mouser Price/Stock" "" (id 9) (at 252.73 58.42 0)
+      (effects (font (size 1.27 1.27)) (justify left) hide)
+    )
+    (property "Arrow Part Number" "" (id 10) (at 252.73 60.96 0)
+      (effects (font (size 1.27 1.27)) (justify left) hide)
+    )
+    (property "Arrow Price/Stock" "" (id 11) (at 252.73 63.5 0)
+      (effects (font (size 1.27 1.27)) (justify left) hide)
+    )
+    (pin "1")
+    (pin "2")
+  )
   (symbol (lib_id "power:GND") (at 207.01 48.26 90) (unit 1)
     (in_bom yes) (on_board yes) (fields_autoplaced)
-    (property "Reference" "#PWR041" (id 0) (at 213.36 48.26 0)
+    (property "Reference" "#PWR039" (id 0) (at 213.36 48.26 0)
       (effects (font (size 1.27 1.27)) hide)
     )
@@
     )
     (pin "1")
+  )
+  (symbol (lib_id "SamacSys_Parts_Power:CC0603KRX7R9BB104") (at 223.52 39.37 90) (unit 1)
+    (in_bom yes) (on_board yes) (fields_autoplaced)
+    (property "Reference" "C13" (id 0) (at 227.33 31.7499 90)
+      (effects (font (size 1.27 1.27)) (justify right))
+    )
+    (property "Value" "CC0603KRX7R9BB104" (id 1) (at 227.33 34.2899 90)
+      (effects (font (size 1.27 1.27)) (justify right))
+    )
+    (property "Footprint" "CAPC1608X90N" (id 2) (at 222.25 30.48 0)
+      (effects (font (size 1.27 1.27)) (justify left) hide)
+    )
+    (property "Datasheet" "http://componentsearchengine.com/Datasheets/3/CC0603KRX7R9BB104.pdf" (id 3) (at 224.79 30.48 0)
+      (effects (font (size 1.27 1.27)) (justify left) hide)
+    )
+    (property "Description" "CAPACITOR, 0603 100nF +/-10% 50V" (id 4) (at 227.33 30.48 0)
+      (effects (font (size 1.27 1.27)) (justify left) hide)
+    )
+    (property "Height" "0.9" (id 5) (at 229.87 30.48 0)
+      (effects (font (size 1.27 1.27)) (justify left) hide)
+    )
+    (property "Manufacturer_Name" "YAGEO (PHYCOMP)" (id 6) (at 232.41 30.48 0)
+      (effects (font (size 1.27 1.27)) (justify left) hide)
+    )
+    (property "Manufacturer_Part_Number" "CC0603KRX7R9BB104" (id 7) (at 234.95 30.48 0)
+      (effects (font (size 1.27 1.27)) (justify left) hide)
+    )
+    (property "Mouser Part Number" "603-CC603KRX7R9BB104" (id 8) (at 237.49 30.48 0)
+      (effects (font (size 1.27 1.27)) (justify left) hide)
+    )
+    (property "Mouser Price/Stock" "https://www.mouser.co.uk/ProductDetail/YAGEO/CC0603KRX7R9BB104?qs=vTakOoo5QyLvVCYM2ge8LQ%3D%3D" (id 9) (at 240.03 30.48 0)
+      (effects (font (size 1.27 1.27)) (justify left) hide)
+    )
+    (property "Arrow Part Number" "CC0603KRX7R9BB104" (id 10) (at 242.57 30.48 0)
+      (effects (font (size 1.27 1.27)) (justify left) hide)
+    )
+    (property "Arrow Price/Stock" "https://www.arrow.com/en/products/cc0603krx7r9bb104/yageo?region=nac" (id 11) (at 245.11 30.48 0)
+      (effects (font (size 1.27 1.27)) (justify left) hide)
+    )
+    (pin "1")
+    (pin "2")
   )
   (symbol (lib_id "power:GND") (at 104.14 140.97 0) (unit 1)
     (in_bom yes) (on_board yes)
-    (property "Reference" "#PWR037" (id 0) (at 104.14 147.32 0)
+    (property "Reference" "#PWR036" (id 0) (at 104.14 147.32 0)
       (effects (font (size 1.27 1.27)) hide)
     )
@@
   (symbol (lib_id "power:GND") (at 152.4 128.27 90) (unit 1)
     (in_bom yes) (on_board yes)
-    (property "Reference" "#PWR039" (id 0) (at 158.75 128.27 0)
+    (property "Reference" "#PWR037" (id 0) (at 158.75 128.27 0)
       (effects (font (size 1.27 1.27)) hide)
     )
@@
   (symbol (lib_id "power:GND") (at 78.74 91.44 0) (unit 1)
     (in_bom yes) (on_board yes) (fields_autoplaced)
-    (property "Reference" "#PWR036" (id 0) (at 78.74 97.79 0)
-      (effects (font (size 1.27 1.27)) hide)
-    )
+    (property "Reference" "#PWR035" (id 0) (at 78.74 97.79 0)
+      (effects (font (size 1.27 1.27)) hide)
+    )
