File: PCB/main/sensing.kicad_sch (KiCad schematic)
At the start: 16 parts, among them IC1 LM358DT

Commit message: gerber files and dat
Parts:
- renumbered TP7 to TP5, TP8 to TP6, TP9 to TP7
Changed lines of the file:
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@@
   (symbol (lib_id "power:GND") (at 158.75 160.02 0) (unit 1)
     (in_bom yes) (on_board yes) (fields_autoplaced)
-    (property "Reference" "#PWR034" (id 0) (at 158.75 166.37 0)
+    (property "Reference" "#PWR033" (id 0) (at 158.75 166.37 0)
       (effects (font (size 1.27 1.27)) hide)
     )
@@
   (symbol (lib_id "power:GND") (at 119.38 151.13 0) (unit 1)
     (in_bom yes) (on_board yes) (fields_autoplaced)
-    (property "Reference" "#PWR033" (id 0) (at 119.38 157.48 0)
+    (property "Reference" "#PWR032" (id 0) (at 119.38 157.48 0)
       (effects (font (size 1.27 1.27)) hide)
     )
@@
   (symbol (lib_id "SamacSys_Parts_power:5017") (at 86.36 133.35 90) (unit 1)
     (in_bom yes) (on_board yes) (fields_autoplaced)
-    (property "Reference" "TP7" (id 0) (at 90.17 121.9199 90)
+    (property "Reference" "TP5" (id 0) (at 90.17 121.9199 90)
       (effects (font (size 1.27 1.27)) (justify right))
     )
@@
   (symbol (lib_id "SamacSys_Parts_power:5017") (at 121.92 133.35 90) (unit 1)
     (in_bom yes) (on_board yes) (fields_autoplaced)
-    (property "Reference" "TP8" (id 0) (at 125.73 121.9199 90)
+    (property "Reference" "TP6" (id 0) (at 125.73 121.9199 90)
       (effects (font (size 1.27 1.27)) (justify right))
     )
@@
   (symbol (lib_id "power:GND") (at 82.55 151.13 0) (unit 1)
     (in_bom yes) (on_board yes) (fields_autoplaced)
-    (property "Reference" "#PWR031" (id 0) (at 82.55 157.48 0)
+    (property "Reference" "#PWR030" (id 0) (at 82.55 157.48 0)
       (effects (font (size 1.27 1.27)) hide)
     )
@@
   (symbol (lib_id "power:GND") (at 25.4 157.48 0) (unit 1)
     (in_bom yes) (on_board yes) (fields_autoplaced)
-    (property "Reference" "#PWR029" (id 0) (at 25.4 163.83 0)
+    (property "Reference" "#PWR028" (id 0) (at 25.4 163.83 0)
       (effects (font (size 1.27 1.27)) hide)
     )
@@
   (symbol (lib_id "SamacSys_Parts_power:5017") (at 154.94 133.35 0) (unit 1)
     (in_bom yes) (on_board yes) (fields_autoplaced)
-    (property "Reference" "TP9" (id 0) (at 171.45 132.0799 0)
+    (property "Reference" "TP7" (id 0) (at 171.45 132.0799 0)
       (effects (font (size 1.27 1.27)) (justify left))
     )
@@
   (symbol (lib_id "power:GND") (at 246.38 130.81 0) (mirror y) (unit 1)
     (in_bom yes) (on_board yes) (fields_autoplaced)
-    (property "Reference" "#PWR035" (id 0) (at 246.38 137.16 0)
+    (property "Reference" "#PWR034" (id 0) (at 246.38 137.16 0)
       (effects (font (size 1.27 1.27)) hide)
     )
@@
   (symbol (lib_id "power:GND") (at 74.93 153.67 0) (unit 1)
     (in_bom yes) (on_board yes) (fields_autoplaced)
-    (property "Reference" "#PWR030" (id 0) (at 74.93 160.02 0)
+    (property "Reference" "#PWR029" (id 0) (at 74.93 160.02 0)
       (effects (font (size 1.27 1.27)) hide)
     )
@@
   (symbol (lib_id "power:GND") (at 111.76 153.67 0) (unit 1)
     (in_bom yes) (on_board yes) (fields_autoplaced)
-    (property "Reference" "#PWR032" (id 0) (at 111.76 160.02 0)
-      (effects (font (size 1.27 1.27)) hide)
-    )
+    (property "Reference" "#PWR031" (id 0) (at 111.76 160.02 0)
+      (effects (font (size 1.27 1.27)) hide)
+    )

Commit message: created BOM
Parts:
- A1, A2: Comment (none) -> Sensor; JLCPCB Part (none) -> C146233; JLCPCB Part Number (none) -> C146233; Price($) (none) -> 0.1407
- C10, C9: Comment (none) -> 1uF; JLCPCB Part Number (none) -> C15849; Price($) (none) -> 0.0055
- IC1: Comment (none) -> LM358DT; JLCPCB Part Number (none) -> C9481; LCSC C9418 -> C9481; Price($) (none) -> 0.1043
- R10, R11, R4, R5, R8, R9: Comment (none) -> 1k; JLCPCB Part Number (none) -> C22548; Price($) (none) -> 0.0013
- R6, R7: Comment (none) -> 536k; JLCPCB Part (none) -> C144748; JLCPCB Part Number (none) -> C144748; Price($) (none) -> 0.0011
- TP5, TP6, TP7: Comment (none) -> test point; JLCPCB Part Number (none) -> C238130; LCSC (none) -> C238130; Price($) (none) -> 0.4796
Changed lines of the file:
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@@
+      (effects (font (size 1.27 1.27)) hide)
+    )
+    (property "Comment" "1k" (id 15) (at 160.02 140.97 0)
+      (effects (font (size 1.27 1.27)) hide)
+    )
+    (property "JLCPCB Part Number" "C22548" (id 16) (at 160.02 140.97 0)
+      (effects (font (size 1.27 1.27)) hide)
+    )
+    (property "Price($)" "0.0013" (id 17) (at 160.02 140.97 0)
       (effects (font (size 1.27 1.27)) hide)
     )
@@
       (effects (font (size 1.27 1.27)) hide)
     )
+    (property "Comment" "1k" (id 15) (at 154.94 114.3 0)
+      (effects (font (size 1.27 1.27)) hide)
+    )
+    (property "JLCPCB Part Number" "C22548" (id 16) (at 154.94 114.3 0)
+      (effects (font (size 1.27 1.27)) hide)
+    )
+    (property "Price($)" "0.0013" (id 17) (at 154.94 114.3 0)
+      (effects (font (size 1.27 1.27)) hide)
+    )
     (pin "1")
     (pin "2")
@@
     )
     (property "MANUFACTURER" "Samsung Electro-Mechanics" (id 14) (at 82.55 133.35 0)
+      (effects (font (size 1.27 1.27)) hide)
+    )
+    (property "Comment" "1uF" (id 15) (at 82.55 133.35 0)
+      (effects (font (size 1.27 1.27)) hide)
+    )
+    (property "JLCPCB Part Number" "C15849" (id 16) (at 82.55 133.35 0)
+      (effects (font (size 1.27 1.27)) hide)
+    )
+    (property "Price($)" "0.0055" (id 17) (at 82.55 133.35 0)
       (effects (font (size 1.27 1.27)) hide)
     )
@@
       (effects (font (size 1.27 1.27)) hide)
     )
+    (property "Comment" "1k" (id 15) (at 158.75 114.3 0)
+      (effects (font (size 1.27 1.27)) hide)
+    )
+    (property "JLCPCB Part Number" "C22548" (id 16) (at 158.75 114.3 0)
+      (effects (font (size 1.27 1.27)) hide)
+    )
+    (property "Price($)" "0.0013" (id 17) (at 158.75 114.3 0)
+      (effects (font (size 1.27 1.27)) hide)
+    )
     (pin "1")
     (pin "2")
@@
       (effects (font (size 1.27 1.27)) hide)
     )
+    (property "Comment" "Sensor" (id 10) (at 68.58 127 0)
+      (effects (font (size 1.27 1.27)) hide)
+    )
+    (property "JLCPCB Part" "C146233" (id 11) (at 68.58 127 0)
+      (effects (font (size 1.27 1.27)) hide)
+    )
+    (property "JLCPCB Part Number" "C146233" (id 12) (at 68.58 127 0)
+      (effects (font (size 1.27 1.27)) hide)
+    )
+    (property "Price($)" "0.1407" (id 13) (at 68.58 127 0)
+      (effects (font (size 1.27 1.27)) hide)
+    )
     (pin "1")
     (pin "2")
@@
       (effects (font (size 1.27 1.27)) hide)
     )
+    (property "Comment" "536k" (id 15) (at 74.93 133.35 0)
+      (effects (font (size 1.27 1.27)) hide)
+    )
+    (property "JLCPCB Part" "C144748" (id 16) (at 74.93 133.35 0)
+      (effects (font (size 1.27 1.27)) hide)
+    )
+    (property "JLCPCB Part Number" "C144748" (id 17) (at 74.93 133.35 0)
+      (effects (font (size 1.27 1.27)) hide)
+    )
+    (property "Price($)" "0.0011" (id 18) (at 74.93 133.35 0)
+      (effects (font (size 1.27 1.27)) hide)
+    )
     (pin "1")
     (pin "2")
@@
       (effects (font (size 1.27 1.27)) hide)
     )
+    (property "Comment" "1k" (id 15) (at 158.75 140.97 0)
+      (effects (font (size 1.27 1.27)) hide)
+    )
+    (property "JLCPCB Part Number" "C22548" (id 16) (at 158.75 140.97 0)
+      (effects (font (size 1.27 1.27)) hide)
+    )
+    (property "Price($)" "0.0013" (id 17) (at 158.75 140.97 0)
+      (effects (font (size 1.27 1.27)) hide)
+    )
     (pin "1")
     (pin "2")
@@
     )
     (property "Price" "$0.1407" (id 9) (at 105.41 127 0)
+      (effects (font (size 1.27 1.27)) hide)
+    )
+    (property "Comment" "Sensor" (id 10) (at 105.41 127 0)
+      (effects (font (size 1.27 1.27)) hide)
+    )
+    (property "JLCPCB Part" "C146233" (id 11) (at 105.41 127 0)
+      (effects (font (size 1.27 1.27)) hide)
+    )
+    (property "JLCPCB Part Number" "C146233" (id 12) (at 105.41 127 0)
+      (effects (font (size 1.27 1.27)) hide)
+    )
+    (property "Price($)" "0.1407" (id 13) (at 105.41 127 0)
       (effects (font (size 1.27 1.27)) hide)
     )
@@
       (effects (font (size 1.27 1.27)) (justify left) hide)
     )
+    (property "Comment" "test point" (id 12) (at 86.36 133.35 0)
+      (effects (font (size 1.27 1.27)) hide)
+    )
+    (property "JLCPCB Part Number" "C238130" (id 13) (at 86.36 133.35 0)
+      (effects (font (size 1.27 1.27)) hide)
+    )
+    (property "LCSC" "C238130" (id 14) (at 86.36 133.35 0)
+      (effects (font (size 1.27 1.27)) hide)
+    )
+    (property "Price($)" "0.4796" (id 15) (at 86.36 133.35 0)
+      (effects (font (size 1.27 1.27)) hide)
+    )
     (pin "1")
   )
@@
       (effects (font (size 1.27 1.27)) (justify left) hide)
     )
+    (property "Comment" "test point" (id 12) (at 121.92 133.35 0)
+      (effects (font (size 1.27 1.27)) hide)
+    )
+    (property "JLCPCB Part Number" "C238130" (id 13) (at 121.92 133.35 0)
+      (effects (font (size 1.27 1.27)) hide)
+    )
+    (property "LCSC" "C238130" (id 14) (at 121.92 133.35 0)
+      (effects (font (size 1.27 1.27)) hide)
+    )
+    (property "Price($)" "0.4796" (id 15) (at 121.92 133.35 0)
+      (effects (font (size 1.27 1.27)) hide)
+    )
     (pin "1")
   )
@@
     (property "Arrow Price/Stock" "" (id 11) (at 171.45 153.67 0)
       (effects (font (size 1.27 1.27)) (justify left) hide)
+    )
+    (property "Comment" "test point" (id 12) (at 154.94 133.35 0)
+      (effects (font (size 1.27 1.27)) hide)
+    )
+    (property "JLCPCB Part Number" "C238130" (id 13) (at 154.94 133.35 0)
+      (effects (font (size 1.27 1.27)) hide)
+    )
+    (property "LCSC" "C238130" (id 14) (at 154.94 133.35 0)
+      (effects (font (size 1.27 1.27)) hide)
+    )
+    (property "Price($)" "0.4796" (id 15) (at 154.94 133.35 0)
+      (effects (font (size 1.27 1.27)) hide)
     )
     (pin "1")
@@
       (effects (font (size 1.27 1.27)) (justify left) hide)
     )
-    (property "LCSC" "C9418" (id 12) (at 217.17 123.19 0)
+    (property "LCSC" "C9481" (id 12) (at 217.17 123.19 0)
       (effects (font (size 1.27 1.27)) hide)
     )
@@
     )
     (property "MANUFACTURER" "STMicroelectronics" (id 14) (at 217.17 123.19 0)
+      (effects (font (size 1.27 1.27)) hide)
+    )
+    (property "Comment" "LM358DT" (id 15) (at 217.17 123.19 0)
+      (effects (font (size 1.27 1.27)) hide)
+    )
+    (property "JLCPCB Part Number" "C9481" (id 16) (at 217.17 123.19 0)
+      (effects (font (size 1.27 1.27)) hide)
+    )
+    (property "Price($)" "0.1043" (id 17) (at 217.17 123.19 0)
       (effects (font (size 1.27 1.27)) hide)
     )
@@
       (effects (font (size 1.27 1.27)) hide)
     )
+    (property "Comment" "1k" (id 15) (at 25.4 134.62 0)
+      (effects (font (size 1.27 1.27)) hide)
+    )
+    (property "JLCPCB Part Number" "C22548" (id 16) (at 25.4 134.62 0)
+      (effects (font (size 1.27 1.27)) hide)
+    )
+    (property "Price($)" "0.0013" (id 17) (at 25.4 134.62 0)
+      (effects (font (size 1.27 1.27)) hide)
+    )
     (pin "1")
     (pin "2")
@@
       (effects (font (size 1.27 1.27)) hide)
     )
+    (property "Comment" "1k" (id 15) (at 25.4 154.94 0)
+      (effects (font (size 1.27 1.27)) hide)
+    )
+    (property "JLCPCB Part Number" "C22548" (id 16) (at 25.4 154.94 0)
+      (effects (font (size 1.27 1.27)) hide)
+    )
+    (property "Price($)" "0.0013" (id 17) (at 25.4 154.94 0)
+      (effects (font (size 1.27 1.27)) hide)
+    )
     (pin "1")
     (pin "2")
@@
       (effects (font (size 1.27 1.27)) hide)
     )
+    (property "Comment" "1uF" (id 15) (at 119.38 133.35 0)
+      (effects (font (size 1.27 1.27)) hide)
+    )
+    (property "JLCPCB Part Number" "C15849" (id 16) (at 119.38 133.35 0)
+      (effects (font (size 1.27 1.27)) hide)
+    )
+    (property "Price($)" "0.0055" (id 17) (at 119.38 133.35 0)
+      (effects (font (size 1.27 1.27)) hide)
+    )
     (pin "1")
     (pin "2")
@@
       (effects (font (size 1.27 1.27)) hide)
     )
+    (property "Comment" "536k" (id 15) (at 111.76 133.35 0)
+      (effects (font (size 1.27 1.27)) hide)
+    )
+    (property "JLCPCB Part" "C144748" (id 16) (at 111.76 133.35 0)
+      (effects (font (size 1.27 1.27)) hide)
+    )
+    (property "JLCPCB Part Number" "C144748" (id 17) (at 111.76 133.35 0)
+      (effects (font (size 1.27 1.27)) hide)
+    )
+    (property "Price($)" "0.0011" (id 18) (at 111.76 133.35 0)
+      (effects (font (size 1.27 1.27)) hide)
+    )

Commit message: new PCB
Parts:
- TP5, TP6, TP7: footprint 5017 -> SamacSys_Parts_Power:5017
Changed lines of the file:
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@@
       (effects (font (size 1.27 1.27)) (justify right))
     )
-    (property "Footprint" "5017" (id 2) (at 83.82 116.84 0)
+    (property "Footprint" "SamacSys_Parts_Power:5017" (id 2) (at 83.82 116.84 0)
       (effects (font (size 1.27 1.27)) (justify left) hide)
     )
@@
       (effects (font (size 1.27 1.27)) (justify right))
     )
-    (property "Footprint" "5017" (id 2) (at 119.38 116.84 0)
+    (property "Footprint" "SamacSys_Parts_Power:5017" (id 2) (at 119.38 116.84 0)
       (effects (font (size 1.27 1.27)) (justify left) hide)
     )
@@
       (effects (font (size 1.27 1.27)) (justify left))
     )
-    (property "Footprint" "5017" (id 2) (at 171.45 130.81 0)
+    (property "Footprint" "SamacSys_Parts_Power:5017" (id 2) (at 171.45 130.81 0)
       (effects (font (size 1.27 1.27)) (justify left) hide)
     )
